Commit message: add imu, orb slam working with gazebo sim

File: src/orbslam_nav_sim/urdf/mobile_base.xacro (robot description, xacro)
@@ -8,4 +8,5 @@
   <xacro:property name="wheel_length" value="0.05"/>
   <xacro:property name="camera_size" value="0.05"/>
+  <xacro:property name="imu_size" value="0.03"/>
   <!-- Link -->
   <link name="base_footprint" />
@@ -78,4 +79,20 @@
     <xacro:box_inertia m="1.0" l="${camera_size}" w="${camera_size}" h="${camera_size}" xyz="0 0 0" rpy="0 0 0" />
   </link>
+  <link name="imu_link">
+    <visual>
+      <geometry>
+        <box size="${imu_size} ${imu_size} ${imu_size}"/>
+      </geometry>
+      <origin xyz="0 0 0" rpy="0 0 0"/>
+      <material name="grey"/>
+    </visual>
+    <collision>
+        <geometry>
+            <box size="${imu_size} ${imu_size} ${imu_size}"/>
+        </geometry>
+        <origin xyz="0.0 0.0 0.0" rpy="0.0 0.0 0.0"/>
+    </collision>
+    <xacro:box_inertia m="1.0" l="${imu_size}" w="${imu_size}" h="${imu_size}" xyz="0 0 0" rpy="0 0 0" />
+  </link>
   <!-- Joint -->
   <joint name="base_joint" type="fixed">
@@ -106,3 +123,8 @@
     <origin xyz="${base_length / 2 - camera_size / 2.0} 0.0 ${base_height + camera_size / 2.0}" rpy="0.0 0.0 0.0"/>
   </joint>
+  <joint name="base_imu_joint" type="fixed">
+    <parent link="base_link"/>
+    <child link="imu_link"/>
+    <origin xyz="0 0.0 ${base_height + imu_size / 2.0}" rpy="0.0 0.0 0.0"/>
+  </joint>
 </robot>

File: src/orbslam_nav_sim/urdf/mobile_base_gazebo.xacro (robot description, xacro)
@@ -42,5 +42,5 @@
       <update_rate>30.0</update_rate>
       <camera name="head">
-        <horizontal_fov>1.3962634</horizontal_fov>
+        <horizontal_fov>1.08</horizontal_fov>
         <image>
           <width>640</width>
@@ -50,5 +50,5 @@
         <clip>
           <near>0.02</near>
-          <far>300</far>
+          <far>100</far>
         </clip>
       </camera>
@@ -63,3 +63,26 @@
     </sensor>
   </gazebo>
+  <!-- IMU -->
+  <gazebo reference="imu_link">
+    <gravity>true</gravity>
+    <sensor name="imu_sensor" type="imu">
+      <always_on>true</always_on>
+      <update_rate>200</update_rate>
+      <visualize>true</visualize>
+      <plugin filename="libgazebo_ros_imu_sensor.so" name="imu_plugin">
+        <ros>
+           <namespace>/</namespace>
+           <remapping>~/out:=imu</remapping>
+        </ros>
+        <topicName>imu</topicName>
+        <bodyName>imu_link</bodyName>
+        <updateRateHZ>200.0</updateRateHZ>
+        <gaussianNoise>0.0</gaussianNoise>
+        <xyzOffset>0 0 0</xyzOffset>
+        <rpyOffset>0 0 0</rpyOffset>
+        <frameName>imu_link</frameName>
+      </plugin>
+      <pose>0 0 0 0 0 0</pose>
+    </sensor>
+  </gazebo>
 </robot>
